Commit message: modify diffbot to work, add imubot

File: diff_drive_controller/test/diffbot.xacro (robot description, xacro)
@@ -21,5 +21,5 @@
     <visual>
       <geometry>
-        <box size="${width} 0.1 0.1"/>
+        <box size="0.1 ${width} 0.1"/>
       </geometry>
     </visual>
@@ -28,5 +28,5 @@
       <origin xyz="0 0 0"/>
       <geometry>
-        <box size="${width} 0.1 0.1"/>
+        <box size="0.1 ${width} 0.1"/>
       </geometry>
     </collision>
@@ -52,9 +52,14 @@
   <!-- Wheels -->
   <wheel name="wheel_0" parent="base" radius="${wheel_radius}" thickness="${thickness}">
-    <origin xyz="${width/2+axel_offset} 0 0" rpy="${-90 * deg_to_rad} 0 0"/>
+    <origin xyz="0 ${width/2+axel_offset} 0" rpy="${-90 * deg_to_rad} 0 0"/>
   </wheel>
   <wheel name="wheel_1" parent="base" radius="${wheel_radius}" thickness="${thickness}">
-    <origin xyz="${-width/2+axel_offset} 0 0" rpy="${-90 * deg_to_rad} 0 0"/>
+    <origin xyz="0 ${-width/2+axel_offset} 0" rpy="${-90 * deg_to_rad} 0 0"/>
   </wheel>
+  <!-- gazebo>
+    <plugin name="gazebo_ros_control" filename="libgazebo_ros_control.so">
+      <robotNamespace></robotNamespace>
+    </plugin>
+  </gazebo -->
   <!-- Colour -->
   <gazebo reference="base_link">

File: diff_drive_controller/test/wheel.xacro (robot description, xacro)
@@ -28,12 +28,20 @@
     </joint>
     <!-- Transmission is important to link the joints and the controller -->
-    <transmission name="${name}_joint_trans" type="SimpleTransmission">
-      <actuator name="${name}_joint_motor"/>
-      <joint name="${name}_joint"/>
-      <mechanicalReduction>1</mechanicalReduction>
-      <motorTorqueConstant>1</motorTorqueConstant>
+    <transmission name="${name}_joint_trans">
+      <type>transmission_interface/SimpleTransmission</type>
+      <joint name="${name}_joint">
+        <hardwareInterface>VelocityJointInterface</hardwareInterface>
+      </joint>
+      <actuator name="${name}_joint_motor">
+        <hardwareInterface>VelocityJointInterface</hardwareInterface>
+        <mechanicalReduction>1</mechanicalReduction>
+        <motorTorqueConstant>1</motorTorqueConstant>
+      </actuator>
     </transmission>
     <gazebo reference="${name}_link">
       <material>Gazebo/Red</material>
+      <selfCollide>true</selfCollide>
+      <mu1 value="0.8" />
+      <mu2 value="0.8" />
     </gazebo>
   </xacro:macro>
